File: StudiokiController/OLEDDisplay.sch (KiCad schematic (older format))
At the start: 8 parts, among them J2 Conn_01x30_Male

Commit message: Added Datasheets
Connections:
- net PIN renamed RES
Changed lines of the file:
@@
 EESchema Schematic File Version 4
+LIBS:StudiokiController-cache
 EELAYER 30 0
 EELAYER END
@@
 	4350 3950 4350 4050
 Text HLabel 5450 3850 0    50   Input ~ 0
-PIN
+RES
 Wire Wire Line
 	5450 3850 5600 3850
