File: StudiokiController/OLEDDisplay.sch (KiCad schematic (older format))
At the start: 8 parts, among them J2 Conn_01x30_Male

Commit message: first PCB
Parts:
- renumbered C6 to C14, C7 to C15, C8 to C16, C9 to C17, C10 to C18, C11 to C19, J2 to J10
Connections:
- net GND: now also C18.2, C19.2
Changed lines of the file:
@@
 EESchema Schematic File Version 4
 LIBS:StudiokiController-cache
-EELAYER 29 0
+EELAYER 30 0
 EELAYER END
 $Descr A4 11693 8268
 encoding utf-8
-Sheet 2 4
+Sheet 2 5
 Title ""
 Date ""
@@
 $EndDescr
 $Comp
-L Connector:Conn_01x30_Male J2
+L Connector:Conn_01x30_Male J10
 U 1 1 5DEA61AC
 P 5800 3950
-F 0 "J2" H 5772 3924 50  0000 R CNN
+F 0 "J10" H 5772 3924 50  0000 R CNN
 F 1 "Conn_01x30_Male" H 5772 3833 50  0000 R CNN
 F 2 "StudiokiController:OLED-solder" H 5800 3950 50  0001 C CNN
@@
 	4350 5350 4350 5450
 $Comp
-L Device:C C6
+L Device:C C14
 U 1 1 5DEAC8A5
 P 4800 5250
-F 0 "C6" V 4548 5250 50  0000 C CNN
+F 0 "C14" V 4548 5250 50  0000 C CNN
 F 1 "2.2uF" V 4639 5250 50  0000 C CNN
 F 2 "Capacitor_SMD:C_0603_1608Metric" H 4838 5100 50  0001 C CNN
@@
 SCL
 $Comp
-L Device:C C7
+L Device:C C15
 U 1 1 5DEAFA24
 P 5100 5150
-F 0 "C7" V 4848 5150 50  0000 C CNN
+F 0 "C15" V 4848 5150 50  0000 C CNN
 F 1 "4.7uF" V 4939 5150 50  0000 C CNN
 F 2 "Capacitor_SMD:C_0603_1608Metric" H 5138 5000 50  0001 C CNN
@@
 	4350 3650 4350 3750
 Wire Wire Line
-	5800 3950 6200 3950
-Wire Wire Line
 	6200 3950 6200 3850
 Connection ~ 6200 3950
@@
 	6200 3950 6550 3950
 $Comp
-L Device:C C10
+L Device:C C18
 U 1 1 5DEB7C5F
 P 6200 3700
-F 0 "C10" H 6315 3746 50  0000 L CNN
+F 0 "C18" H 6315 3746 50  0000 L CNN
 F 1 "1uF" H 6315 3655 50  0000 L CNN
 F 2 "Capacitor_SMD:C_0603_1608Metric" H 6238 3550 50  0001 C CNN
@@
 $EndComp
 $Comp
-L Device:C C11
+L Device:C C19
 U 1 1 5DEB83BE
 P 6550 3700
-F 0 "C11" H 6665 3746 50  0000 L CNN
+F 0 "C19" H 6665 3746 50  0000 L CNN
 F 1 "1uF" H 6665 3655 50  0000 L CNN
 F 2 "Capacitor_SMD:C_0603_1608Metric" H 6588 3550 50  0001 C CNN
@@
 	4350 3250 4350 3450
 $Comp
-L Device:C C8
+L Device:C C16
 U 1 1 5DEC0A3E
 P 5350 2950
-F 0 "C8" V 5602 2950 50  0000 C CNN
+F 0 "C16" V 5602 2950 50  0000 C CNN
 F 1 "1uF" V 5511 2950 50  0000 C CNN
 F 2 "Capacitor_SMD:C_0603_1608Metric" H 5388 2800 50  0001 C CNN
@@
 	5200 2850 5600 2850
 $Comp
-L Device:C C9
+L Device:C C17
 U 1 1 5DEC3994
 P 6100 2750
-F 0 "C9" V 6352 2750 50  0000 C CNN
+F 0 "C17" V 6352 2750 50  0000 C CNN
 F 1 "1uF" V 6261 2750 50  0000 C CNN
 F 2 "Capacitor_SMD:C_0603_1608Metric" H 6138 2600 50  0001 C CNN
@@
 Text HLabel 6550 3050 2    50   Input ~ 0
 3V3
+Wire Wire Line
+	5600 3950 6200 3950
+Connection ~ 5600 3950
 $EndSCHEMATC
