File: StudiokiController/StudiokiController.sch (KiCad schematic (older format))
At the start: 31 parts, among them J1 USB_B_Mini, J3 Conn_01x04_Male, J4 57PC5FS, J5 Conn_01x02_Female, J6 Screw_Terminal_01x03, J7 WJ142R-5.08-3P, Q1 Q_DUAL_NPN_NPN_E1B1C2E2B2C1, SW1 SW_Push, SW2 SW_Push, SW3 SW_Push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

Commit message: first PCB
Parts:
- removed J3: Conn_01x04_Male, Connector_PinHeader_2.54mm:PinHeader_1x04_P2.54mm_Vertical, symbol Connector:Conn_01x04_Male
- removed J6: Screw_Terminal_01x03, WJ142R-5.08-3P:RHDR6W120P762X508_2X3_1524X1410X1355P, symbol Connector:Screw_Terminal_01x03
- removed R10, R11, R8, R9: 100, Resistor_SMD:R_0603_1608Metric, symbol Device:R
- added C10, C11, C13, C6, C7: 100nF, Capacitor_SMD:C_0603_1608Metric, symbol Device:C
- added C8, C9: 10uF tantal, Capacitor_Tantalum_SMD:CP_EIA-3216-12_Kemet-S, symbol Device:CP1_Small
- added D5, D6, D7: LED, LED_SMD:LED_0603_1608Metric, symbol Device:LED
- added J2, J6: WJ142R-5.08-3P, RHDR6W120P762X508_2X3_1524X1410X1355P, symbol WJ142R-5.08-3P:WJ142R-5.08-3P
- added J3, J8, J9: Conn_01x04_Female, Connector_PinHeader_2.54mm:PinHeader_1x04_P2.54mm_Vertical, symbol Connector:Conn_01x04_Female
- added U4: AZ1117-3.3, Package_TO_SOT_SMD:SOT-223, symbol Regulator_Linear:AZ1117-3.3
- C12: value 0.1uF -> 100nF
- SW1, SW2, SW3: footprint StudiokiController:TSA063G50250 -> Button_Switch_SMD:SW_SPST_PTS645
Connections:
- net labels added: LED1, LED2, LED3, PE, RELAY3
- net labels removed: MTCK, MTDI, MTDO, MTMS
- wire segments 75 -> 139
Other:
- moved on the sheet: C12, J4, J5, J7, SW1, SW2, SW3, U3

Commit message: New Layout
Parts:
- removed J2, J6, J7: WJ142R-5.08-3P, RHDR6W120P762X508_2X3_1524X1410X1355P, symbol WJ142R-5.08-3P:WJ142R-5.08-3P
- added H1, H2, H3, H4: MountingHole, MountingHole:MountingHole_3.2mm_M3_Pad_Via, symbol Mechanical:MountingHole
- added J10: Conn_01x10_Male, Connector_IDC:IDC-Header_2x05_P2.54mm_Vertical, symbol Connector:Conn_01x10_Male
- added J11, J2, J6, J7: Screw_Terminal_01x03, TerminalBlock_Phoenix:TerminalBlock_Phoenix_PT-1,5-3-5.0-H_1x03_P5.00mm_Horizontal, symbol Connector:Screw_Terminal_01x03
- added J12: Screw_Terminal_01x02, TerminalBlock_Phoenix:TerminalBlock_Phoenix_PT-1,5-2-5.0-H_1x02_P5.00mm_Horizontal, symbol Connector:Screw_Terminal_01x02
- added R10, R7, R9: 100, Resistor_SMD:R_0603_1608Metric, symbol Device:R
- added RV1: MOV-07D391KTR, Varistor:RV_Disc_D7mm_W4.5mm_P5mm, symbol Device:Varistor
- J3, J8, J9: footprint Connector_PinHeader_2.54mm:PinHeader_1x04_P2.54mm_Vertical -> Connector_PinSocket_2.54mm:PinSocket_1x04_P2.54mm_Vertical
Connections:
- net DISP_RES is gone; now on net SW1: U2.26 (IO4)
- net +3V3: now also J10.1 (Pin_1)
- net 230V-N: now also J2.3 (Pin_3), RV1.1
- net 230V-Relay/OUTPUT-A: now also J6.3 (Pin_3)
- net 230V-Relay/OUTPUT-B: now also J6.2 (Pin_2)
- net EN: now also J10.2 (Pin_2)
- net GND: now also J10.9 (Pin_9), J12.2 (Pin_2), R10.1, R7.1, R9.1; no longer D5.1 (K), D6.1 (K), D7.1 (K)
- net IO0: now also J10.3 (Pin_3)
- net RELAY1: now also U2.12 (IO27); no longer U2.11 (IO26)
- net RELAY2: now also U2.11 (IO26); no longer U2.12 (IO27)
- net SCL: now also J10.5 (Pin_5)
- net SDA: now also J10.6 (Pin_6)
- net SW1: now also J10.7 (Pin_7); no longer U2.37 (IO23)
- net SW2: now also U2.27 (IO16), J10.8 (Pin_8); no longer U2.30 (IO18)
- net SW3: now also U2.28 (IO17), J10.10 (Pin_10); no longer U2.31 (IO19)
- net sheet5DF376A8/OUTPUT-A: now also J11.3 (Pin_3)
- net DOOR: now reaches U2.14 (IO12)
- net DOOR: now also J12.1 (Pin_1)
- net IO2: now reaches U2.24 (IO2)
- net IO2: now also J10.4 (Pin_4)
- net at F1.2: now also J2.2 (Pin_2), RV1.2
- new net: D5.1 (K), R7.2
- new net: D6.1 (K), R9.2
- new net: D7.1 (K), R10.2
- new net sheet5DF376A8/OUTPUT-B: J11.2 (Pin_2)
- new net sheet5DF55D65/OUTPUT-A: J7.3 (Pin_3)
- new net sheet5DF55D65/OUTPUT-B: J7.2 (Pin_2)
- no-connect marks 0 -> 28
Other:
- moved on the sheet: D5, D6, D7
