File: StudiokiController/StudiokiController.sch (KiCad schematic (older format))
At the start: 60 parts, among them J1 USB_B_Mini, J10 Conn_01x10_Male, J11 Screw_Terminal_01x03, J12 Screw_Terminal_01x02, J2 Screw_Terminal_01x03, J3 Conn_01x04_Female, J4 57PC5FS, J5 Conn_01x02_Female, J6 Screw_Terminal_01x03, J7 Screw_Terminal_01x03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

Commit message: -
Parts:
- removed JP4: SolderJumper_2_Open, symbol Jumper:SolderJumper_2_Open
- C14, C15, C16: footprint (none) -> Capacitor_SMD:C_0603_1608Metric
- R11: footprint (none) -> Resistor_SMD:R_0603_1608Metric
Connections:
- net at C16.1, JP2.1 (A), U5.10 (RTDIN+): now also J8.2 (Pin_2); no longer J8.3 (Pin_3)
- net at JP1.1 (A), JP2.2 (B), U5.8 (FORCE+): now also J8.3 (Pin_3); no longer J8.2 (Pin_2)
- net SPI_SS renamed CS_K1
Changed lines of the file:
@@
 Text GLabel 10300 5700 2    50   Output ~ 0
 SPI_SCK
-Text GLabel 10300 6000 2    50   Output ~ 0
-SPI_SS
+Text GLabel 10300 6000 2    50   Input ~ 0
+CS_K1
 $Comp
 L Device:C C12
@@
 Text GLabel 1650 3250 0    50   Input ~ 0
 SPI_SCK
-Text GLabel 2850 2250 2    50   Input ~ 0
-SPI_SS
+Text GLabel 2850 2250 2    50   Output ~ 0
+CS_K1
 $Comp
 L SamacSys_Parts:57PC5FS J4
@@
 F 0 "C16" H 6142 3646 50  0000 L CNN
 F 1 "C_Small" H 5900 3400 50  0000 L CNN
-F 2 "" H 6050 3600 50  0001 C CNN
+F 2 "Capacitor_SMD:C_0603_1608Metric" H 6050 3600 50  0001 C CNN
 F 3 "~" H 6050 3600 50  0001 C CNN
 	1    6050 3600
@@
 F 0 "R11" V 5554 2900 50  0000 C CNN
 F 1 "R_Small" V 5650 2900 50  0000 C CNN
-F 2 "" H 5750 2900 50  0001 C CNN
+F 2 "Resistor_SMD:R_0603_1608Metric" H 5750 2900 50  0001 C CNN
 F 3 "~" H 5750 2900 50  0001 C CNN
 	1    5750 2900
@@
 F 0 "C15" H 5292 2596 50  0000 L CNN
 F 1 "C_Small" H 5050 2350 50  0000 L CNN
-F 2 "" H 5200 2550 50  0001 C CNN
+F 2 "Capacitor_SMD:C_0603_1608Metric" H 5200 2550 50  0001 C CNN
 F 3 "~" H 5200 2550 50  0001 C CNN
 	1    5200 2550
@@
 F 0 "C14" H 4892 2596 50  0000 L CNN
 F 1 "C_Small" H 4650 2350 50  0000 L CNN
-F 2 "" H 4800 2550 50  0001 C CNN
+F 2 "Capacitor_SMD:C_0603_1608Metric" H 4800 2550 50  0001 C CNN
 F 3 "~" H 4800 2550 50  0001 C CNN
 	1    4800 2550
@@
 Wire Wire Line
 	5600 3100 5600 3200
-$Comp
-L Jumper:SolderJumper_2_Open JP4
-U 1 1 5DFC7168
-P 6600 2700
-F 0 "JP4" H 6600 2475 50  0000 C CNN
-F 1 "SolderJumper_2_Open" H 6600 2566 50  0000 C CNN
-F 2 "" H 6600 2700 50  0001 C CNN
-F 3 "~" H 6600 2700 50  0001 C CNN
-	1    6600 2700
-	-1   0    0    1
-$EndComp
 Wire Wire Line
 	5900 3300 5900 3400
@@
 	5950 3500 6050 3500
 Wire Wire Line
-	6050 3500 6350 3500
-Wire Wire Line
-	6350 3500 6350 3450
-Wire Wire Line
-	6350 3450 6400 3450
+	6050 3500 6200 3500
+Wire Wire Line
+	6200 3500 6200 3550
+Wire Wire Line
+	6200 3550 6400 3550
 Connection ~ 6050 3500
 Wire Wire Line
-	6250 3550 6400 3550
-Wire Wire Line
-	6250 3400 6250 3550
+	6400 3450 6250 3450
+Wire Wire Line
+	6250 3450 6250 3400
 $EndSCHEMATC

Commit message: -
Parts:
- removed J1: USB_B_Mini, Connector_USB:USB_Micro-B_Molex-105017-0001, symbol Connector:USB_B_Mini
- added J?: USB_B_Micro, symbol Connector:USB_B_Micro
- J4: footprint 57PC5FS -> JanSquare:57PC5FS
- PS1: footprint CONV_RAC03-12SK -> JanSquare:CONV_RAC03-12SK
Connections:
- net GND: now also J?.5 (GND), J?.6 (Shield)
- net at C3.2, U1.16 (VCC): now also J?.1 (VBUS)
- net at U1.6 (UD-): now also J?.2 (D-)
- net at U1.5 (UD+): now also J?.3 (D+)
Changed lines of the file:
@@
 $EndDescr
-$Comp
-L Connector:USB_B_Mini J1
-U 1 1 5DE8582A
-P 950 6700
-F 0 "J1" H 1007 7167 50  0000 C CNN
-F 1 "USB_B_Mini" H 1007 7076 50  0000 C CNN
-F 2 "Connector_USB:USB_Micro-B_Molex-105017-0001" H 1100 6650 50  0001 C CNN
-F 3 "~" H 1100 6650 50  0001 C CNN
-	1    950  6700
-	1    0    0    -1
-$EndComp
 $Comp
 L Interface_USB:CH340G U1
@@
 F 0 "J4" V 9746 5978 50  0000 L CNN
 F 1 "57PC5FS" V 9655 5978 50  0000 L CNN
-F 2 "57PC5FS" H 10300 5950 50  0001 L CNN
+F 2 "JanSquare:57PC5FS" H 10300 5950 50  0001 L CNN
 F 3 "https://componentsearchengine.com/Datasheets/1/57PC5FS.pdf" H 10300 5850 50  0001 L CNN
 F 4 "DIN Connectors DIN CON 5 PIN" H 10300 5750 50  0001 L CNN "Description"
@@
 F 0 "PS1" H 6050 1617 50  0000 C CNN
 F 1 "RAC03-12SK" H 6050 1526 50  0000 C CNN
-F 2 "CONV_RAC03-12SK" H 6050 1150 50  0001 L BNN
+F 2 "JanSquare:CONV_RAC03-12SK" H 6050 1150 50  0001 L BNN
 F 3 "" H 6050 1150 50  0001 L BNN
 F 4 "Recom Power" H 6050 1150 50  0001 L BNN "Field4"
@@
 Wire Wire Line
 	6250 3450 6250 3400
+$Comp
+L Connector:USB_B_Micro J?
+U 1 1 5DF859F8
+P 950 6700
+F 0 "J?" H 1007 7167 50  0000 C CNN
+F 1 "USB_B_Micro" H 1007 7076 50  0000 C CNN
+F 2 "" H 1100 6650 50  0001 C CNN
+F 3 "~" H 1100 6650 50  0001 C CNN
+	1    950  6700
+	1    0    0    -1
+$EndComp
 $EndSCHEMATC

Commit message: -
Parts:
- F1: footprint StudiokiController:Littelfuse65800001009 -> JanSquare:Littelfuse65800001009
- gave numbers to parts that had none: 1
Connections:
- net 230V-L: now also J2.2 (Pin_2), RV1.1; no longer F1.1
- net 230V-N: now also F1.1, F1.2, RV1.2; no longer RV1.1
Other:
- moved on the sheet: F1
Changed lines of the file:
@@
 L Device:Fuse F1
 U 1 1 5DED5CF4
-P 4950 950
-F 0 "F1" V 4753 950 50  0000 C CNN
-F 1 "Fuse" V 4844 950 50  0000 C CNN
-F 2 "StudiokiController:Littelfuse65800001009" V 4880 950 50  0001 C CNN
-F 3 "~" H 4950 950 50  0001 C CNN
-	1    4950 950
+P 4900 750
+F 0 "F1" V 4703 750 50  0000 C CNN
+F 1 "Fuse" V 4794 750 50  0000 C CNN
+F 2 "JanSquare:Littelfuse65800001009" V 4830 750 50  0001 C CNN
+F 3 "~" H 4900 750 50  0001 C CNN
+	1    4900 750
 	0    1    1    0
 $EndComp
@@
 Wire Wire Line
 	4950 1150 4950 1100
-Wire Wire Line
-	4950 1100 5250 1100
 $Comp
 L RAC03-12SK:RAC03-12SK PS1
@@
 	1    0    0    -1
 $EndComp
-Wire Wire Line
-	5100 950  5150 950
 Text GLabel 5150 1150 3    50   UnSpc ~ 0
 230V-L
@@
 $EndComp
 Wire Wire Line
-	4450 1100 4800 1100
-Wire Wire Line
-	4450 1000 4500 1000
+	4450 1100 4500 1100
 Wire Wire Line
 	4800 1000 4800 950
-Wire Wire Line
-	4500 1250 4500 1000
-Connection ~ 4500 1000
-Wire Wire Line
-	4500 1000 4800 1000
-Wire Wire Line
-	4800 1250 4800 1100
-Connection ~ 4800 1100
-Wire Wire Line
-	4800 1100 4950 1100
 $Comp
 L Connector:Screw_Terminal_01x02 J12
@@
 	6250 3450 6250 3400
 $Comp
-L Connector:USB_B_Micro J?
+L Connector:USB_B_Micro J1
 U 1 1 5DF859F8
 P 950 6700
-F 0 "J?" H 1007 7167 50  0000 C CNN
+F 0 "J1" H 1007 7167 50  0000 C CNN
 F 1 "USB_B_Micro" H 1007 7076 50  0000 C CNN
 F 2 "" H 1100 6650 50  0001 C CNN
@@
 	1    0    0    -1
 $EndComp
+Wire Wire Line
+	4800 950  5150 950
+Wire Wire Line
+	4750 750  4650 750
+Wire Wire Line
+	4650 750  4650 1100
+Connection ~ 4650 1100
+Wire Wire Line
+	4950 1100 5250 1100
+Wire Wire Line
+	5050 750  5050 850
+Wire Wire Line
+	4450 1000 4800 1000
+Wire Wire Line
+	4800 1250 4800 1000
+Connection ~ 4800 1000
+Wire Wire Line
+	4500 1100 4500 1250
+Connection ~ 4500 1100
+Wire Wire Line
+	4500 1100 4650 1100
+Wire Wire Line
+	4650 1100 4750 1100
+Wire Wire Line
+	4750 850  4750 1100
+Wire Wire Line
+	4750 850  5050 850
+Connection ~ 4750 1100
+Wire Wire Line
+	4750 1100 4950 1100
 $EndSCHEMATC

Commit message: gjkl
fh
Parts:
- removed C14, C15, C16: C_Small, Capacitor_SMD:C_0603_1608Metric, symbol Device:C_Small
- removed J11: Screw_Terminal_01x03, TerminalBlock_Phoenix:TerminalBlock_Phoenix_PT-1,5-3-5.0-H_1x03_P5.00mm_Horizontal, symbol Connector:Screw_Terminal_01x03
- removed J8: Conn_01x03_Female, StudiokiController:WAGO2060-473-998-404, symbol Connector:Conn_01x03_Female
- removed JP1, JP2, JP3: SolderJumper_2_Open, Jumper:SolderJumper-2_P1.3mm_Open_RoundedPad1.0x1.5mm, symbol Jumper:SolderJumper_2_Open
- removed R11: R_Small, Resistor_SMD:R_0603_1608Metric, symbol Device:R_Small
- removed U5: MAX31865AAP+T, SOP65P777X199-20N, symbol MAX31865AAP_T:MAX31865AAP+T
- J1: footprint (none) -> Connector_USB:USB_Micro-B_Molex-105017-0001
Connections:
- no-connect marks 29 -> 27
Other:
- moved on the sheet: C7, C8, C9, U4
