File: StudiokiController/230V-Relay.sch (KiCad schematic (older format))
At the start: 5 parts, among them Q2 PMV20XNE

Commit message: New Layout
Connections:
- net +12V renamed 12V
Changed lines of the file:
@@
 $Descr A4 11693 8268
 encoding utf-8
-Sheet 5 5
+Sheet 2 4
 Title ""
 Date ""
@@
 AR Path="/5DF55D6C/5DF31335" Ref="RLA2"  Part="1"
 AR Path="/5DF376BF/5DF31335" Ref="RLA3"  Part="1"
-F 0 "RLA3" V 5197 3228 60  0000 L CNN
+F 0 "RLA1" V 5197 3228 60  0000 L CNN
 F 1 "OJE-SH-112HM_000" V 5303 3228 60  0000 L CNN
 F 2 "StudiokiController:OJE-SH-112HM_000" H 5250 3240 60  0001 C CNN
@@
 	0    1    1    0
 $EndComp
-Wire Wire Line
-	6450 1950 5500 1950
 $Comp
 L Device:Q_NMOS_GSD Q?
@@
 AR Path="/5DF55D6C/5DF3133E" Ref="Q3"  Part="1"
 AR Path="/5DF376BF/5DF3133E" Ref="Q4"  Part="1"
-F 0 "Q4" H 4406 3596 50  0000 L CNN
+F 0 "Q2" H 4406 3596 50  0000 L CNN
 F 1 "PMV20XNE" H 4406 3505 50  0000 L CNN
 F 2 "Package_TO_SOT_SMD:SOT-23" H 4400 3650 50  0001 C CNN
@@
 AR Path="/5DF55D6C/5DF31344" Ref="R13"  Part="1"
 AR Path="/5DF376BF/5DF31344" Ref="R8"  Part="1"
-F 0 "R8" H 3970 3896 50  0000 L CNN
+F 0 "R12" H 3970 3896 50  0000 L CNN
 F 1 "10k" H 3970 3805 50  0000 L CNN
 F 2 "Resistor_SMD:R_0603_1608Metric" V 3830 3850 50  0001 C CNN
@@
 	3900 4000 4300 4000
 Wire Wire Line
-	4300 4000 4300 3750
-$Comp
-L power:GND #PWR?
-U 1 1 5DF3134E
-P 4300 4000
-AR Path="/5DF3134E" Ref="#PWR?"  Part="1"
-AR Path="/5DF2D1A8/5DF3134E" Ref="#PWR0111"  Part="1"
-AR Path="/5DF3EB9E/5DF3134E" Ref="#PWR?"  Part="1"
-AR Path="/5DF55D6C/5DF3134E" Ref="#PWR0114"  Part="1"
-AR Path="/5DF376BF/5DF3134E" Ref="#PWR0129"  Part="1"
-F 0 "#PWR0129" H 4300 3750 50  0001 C CNN
-F 1 "GND" H 4305 3827 50  0000 C CNN
-F 2 "" H 4300 4000 50  0001 C CNN
-F 3 "" H 4300 4000 50  0001 C CNN
-	1    4300 4000
-	1    0    0    -1
-$EndComp
-Connection ~ 4300 4000
+	4300 4000 4300 3900
 $Comp
 L Device:LED D?
@@
 AR Path="/5DF55D6C/5DF31355" Ref="D3"  Part="1"
 AR Path="/5DF376BF/5DF31355" Ref="D8"  Part="1"
-F 0 "D8" V 3639 3633 50  0000 R CNN
+F 0 "D1" V 3639 3633 50  0000 R CNN
 F 1 "LED" V 3548 3633 50  0000 R CNN
 F 2 "LED_SMD:LED_0603_1608Metric" H 3600 3750 50  0001 C CNN
@@
 AR Path="/5DF55D6C/5DF3135B" Ref="#PWR0115"  Part="1"
 AR Path="/5DF376BF/5DF3135B" Ref="#PWR0130"  Part="1"
-F 0 "#PWR0130" H 3600 3650 50  0001 C CNN
+F 0 "#PWR0115" H 3600 3650 50  0001 C CNN
 F 1 "GND" H 3605 3727 50  0000 C CNN
 F 2 "" H 3600 3900 50  0001 C CNN
@@
 Connection ~ 3600 3550
 $Comp
-L power:+12V #PWR?
-U 1 1 5DF3136D
-P 5000 1950
-AR Path="/5DF3136D" Ref="#PWR?"  Part="1"
-AR Path="/5DF2D1A8/5DF3136D" Ref="#PWR0113"  Part="1"
-AR Path="/5DF3EB9E/5DF3136D" Ref="#PWR?"  Part="1"
-AR Path="/5DF55D6C/5DF3136D" Ref="#PWR0116"  Part="1"
-AR Path="/5DF376BF/5DF3136D" Ref="#PWR0131"  Part="1"
-F 0 "#PWR0131" H 5000 1800 50  0001 C CNN
-F 1 "+12V" V 5015 2078 50  0000 L CNN
-F 2 "" H 5000 1950 50  0001 C CNN
-F 3 "" H 5000 1950 50  0001 C CNN
-	1    5000 1950
-	0    1    1    0
-$EndComp
-Wire Wire Line
-	4300 3350 4600 3350
-Wire Wire Line
-	4750 3350 4750 3550
-Wire Wire Line
-	4750 3550 5000 3550
-Wire Wire Line
-	5000 2050 4600 2050
-Wire Wire Line
-	4600 2050 4600 2550
-$Comp
 L Device:D D?
 U 1 1 5DF3137A
@@
 AR Path="/5DF55D6C/5DF3137A" Ref="D4"  Part="1"
 AR Path="/5DF376BF/5DF3137A" Ref="D9"  Part="1"
-F 0 "D9" V 4554 2779 50  0000 L CNN
+F 0 "D2" V 4554 2779 50  0000 L CNN
 F 1 "1N4148W-TP" V 4645 2779 50  0000 L CNN
 F 2 "Diode_SMD:D_SOD-123" H 4600 2700 50  0001 C CNN
@@
 $EndComp
 Wire Wire Line
-	4600 2850 4600 3350
-Connection ~ 4600 3350
+	4600 2850 4600 3300
 Wire Wire Line
 	4600 3350 4750 3350
 Text HLabel 3500 3550 0    50   Input ~ 0
 INPUT-3V3
-Text HLabel 5400 3550 2    50   Output ~ 0
+Text HLabel 5550 3650 2    50   Output ~ 0
 OUTPUT-A
-Text HLabel 6450 1950 2    50   Output ~ 0
+Text HLabel 5600 1700 2    50   Output ~ 0
 OUTPUT-B
-Text HLabel 4300 4000 2    50   UnSpc ~ 0
+Text HLabel 4500 3900 2    50   UnSpc ~ 0
 GND
-Text HLabel 5000 1950 0    50   UnSpc ~ 0
+Text HLabel 4950 1650 0    50   UnSpc ~ 0
 12V
 Wire Wire Line
-	5000 2050 5000 1950
-Connection ~ 5000 1950
+	4500 3900 4300 3900
+Connection ~ 4300 3900
+Wire Wire Line
+	4300 3900 4300 3750
+Wire Wire Line
+	4300 3350 4300 3300
+Wire Wire Line
+	4300 3300 4600 3300
+Connection ~ 4600 3300
+Wire Wire Line
+	4600 3300 4600 3350
+Wire Wire Line
+	5000 3550 5000 3600
+Wire Wire Line
+	5000 3600 4750 3600
+Wire Wire Line
+	4750 3350 4750 3600
+Wire Wire Line
+	5400 3550 5400 3650
+Wire Wire Line
+	5400 3650 5550 3650
+Wire Wire Line
+	4950 1650 5000 1650
+Wire Wire Line
+	5000 1650 5000 1850
+Wire Wire Line
+	5000 1850 4600 1850
+Wire Wire Line
+	4600 1850 4600 2550
+Connection ~ 5000 1850
+Wire Wire Line
+	5000 1850 5000 1950
+Wire Wire Line
+	5500 1950 5500 1700
+Wire Wire Line
+	5500 1700 5600 1700
 $EndSCHEMATC
