File: StudiokiController/230V-Relay.sch (KiCad schematic (older format))
At the start: 5 parts, among them Q2 PMV20XNE

Commit message: -
Changed lines of the file:
@@
 AR Path="/5DF55D6C/5DF31335" Ref="RLA2"  Part="1"
 AR Path="/5DF376BF/5DF31335" Ref="RLA3"  Part="1"
-F 0 "RLA2" V 5197 3228 60  0000 L CNN
+F 0 "RLA1" V 5197 3228 60  0000 L CNN
 F 1 "OJE-SH-112HM_000" V 5303 3228 60  0000 L CNN
 F 2 "StudiokiController:OJE-SH-112HM_000" H 5250 3240 60  0001 C CNN
@@
 AR Path="/5DF55D6C/5DF3133E" Ref="Q3"  Part="1"
 AR Path="/5DF376BF/5DF3133E" Ref="Q4"  Part="1"
-F 0 "Q3" H 4406 3596 50  0000 L CNN
+F 0 "Q2" H 4406 3596 50  0000 L CNN
 F 1 "PMV20XNE" H 4406 3505 50  0000 L CNN
 F 2 "Package_TO_SOT_SMD:SOT-23" H 4400 3650 50  0001 C CNN
@@
 AR Path="/5DF55D6C/5DF31344" Ref="R13"  Part="1"
 AR Path="/5DF376BF/5DF31344" Ref="R8"  Part="1"
-F 0 "R13" H 3970 3896 50  0000 L CNN
+F 0 "R12" H 3970 3896 50  0000 L CNN
 F 1 "10k" H 3970 3805 50  0000 L CNN
 F 2 "Resistor_SMD:R_0603_1608Metric" V 3830 3850 50  0001 C CNN
@@
 AR Path="/5DF55D6C/5DF31355" Ref="D3"  Part="1"
 AR Path="/5DF376BF/5DF31355" Ref="D8"  Part="1"
-F 0 "D3" V 3639 3633 50  0000 R CNN
+F 0 "D1" V 3639 3633 50  0000 R CNN
 F 1 "LED" V 3548 3633 50  0000 R CNN
 F 2 "LED_SMD:LED_0603_1608Metric" H 3600 3750 50  0001 C CNN
@@
 AR Path="/5DF55D6C/5DF3135B" Ref="#PWR0115"  Part="1"
 AR Path="/5DF376BF/5DF3135B" Ref="#PWR0130"  Part="1"
-F 0 "#PWR0115" H 3600 3650 50  0001 C CNN
+F 0 "#PWR0112" H 3600 3650 50  0001 C CNN
 F 1 "GND" H 3605 3727 50  0000 C CNN
 F 2 "" H 3600 3900 50  0001 C CNN
@@
 AR Path="/5DF55D6C/5DF3137A" Ref="D4"  Part="1"
 AR Path="/5DF376BF/5DF3137A" Ref="D9"  Part="1"
-F 0 "D4" V 4554 2779 50  0000 L CNN
+F 0 "D2" V 4554 2779 50  0000 L CNN
 F 1 "1N4148W-TP" V 4645 2779 50  0000 L CNN
 F 2 "Diode_SMD:D_SOD-123" H 4600 2700 50  0001 C CNN

Commit message: -
Parts:
- RLA1: footprint StudiokiController:OJE-SH-112HM_000 -> JanSquare::OJE-SH-112HM_000
Changed lines of the file:
@@
 $Descr A4 11693 8268
 encoding utf-8
-Sheet 2 4
+Sheet 3 4
 Title ""
 Date ""
@@
 AR Path="/5DF55D6C/5DF31335" Ref="RLA2"  Part="1"
 AR Path="/5DF376BF/5DF31335" Ref="RLA3"  Part="1"
-F 0 "RLA1" V 5197 3228 60  0000 L CNN
+F 0 "RLA3" V 5197 3228 60  0000 L CNN
 F 1 "OJE-SH-112HM_000" V 5303 3228 60  0000 L CNN
-F 2 "StudiokiController:OJE-SH-112HM_000" H 5250 3240 60  0001 C CNN
+F 2 "JanSquare::OJE-SH-112HM_000" H 5250 3240 60  0001 C CNN
 F 3 "" H 5250 2750 60  0000 C CNN
 	1    5250 2750
@@
 AR Path="/5DF55D6C/5DF3133E" Ref="Q3"  Part="1"
 AR Path="/5DF376BF/5DF3133E" Ref="Q4"  Part="1"
-F 0 "Q2" H 4406 3596 50  0000 L CNN
+F 0 "Q4" H 4406 3596 50  0000 L CNN
 F 1 "PMV20XNE" H 4406 3505 50  0000 L CNN
 F 2 "Package_TO_SOT_SMD:SOT-23" H 4400 3650 50  0001 C CNN
@@
 AR Path="/5DF55D6C/5DF31344" Ref="R13"  Part="1"
 AR Path="/5DF376BF/5DF31344" Ref="R8"  Part="1"
-F 0 "R12" H 3970 3896 50  0000 L CNN
+F 0 "R8" H 3970 3896 50  0000 L CNN
 F 1 "10k" H 3970 3805 50  0000 L CNN
 F 2 "Resistor_SMD:R_0603_1608Metric" V 3830 3850 50  0001 C CNN
@@
 AR Path="/5DF55D6C/5DF31355" Ref="D3"  Part="1"
 AR Path="/5DF376BF/5DF31355" Ref="D8"  Part="1"
-F 0 "D1" V 3639 3633 50  0000 R CNN
+F 0 "D8" V 3639 3633 50  0000 R CNN
 F 1 "LED" V 3548 3633 50  0000 R CNN
 F 2 "LED_SMD:LED_0603_1608Metric" H 3600 3750 50  0001 C CNN
@@
 AR Path="/5DF55D6C/5DF3135B" Ref="#PWR0115"  Part="1"
 AR Path="/5DF376BF/5DF3135B" Ref="#PWR0130"  Part="1"
-F 0 "#PWR0112" H 3600 3650 50  0001 C CNN
+F 0 "#PWR0130" H 3600 3650 50  0001 C CNN
 F 1 "GND" H 3605 3727 50  0000 C CNN
 F 2 "" H 3600 3900 50  0001 C CNN
@@
 AR Path="/5DF55D6C/5DF3137A" Ref="D4"  Part="1"
 AR Path="/5DF376BF/5DF3137A" Ref="D9"  Part="1"
-F 0 "D2" V 4554 2779 50  0000 L CNN
+F 0 "D9" V 4554 2779 50  0000 L CNN
 F 1 "1N4148W-TP" V 4645 2779 50  0000 L CNN
 F 2 "Diode_SMD:D_SOD-123" H 4600 2700 50  0001 C CNN
