File: StudiokiController/StudiokiController.kicad_pcb (KiCad board)
At the start: 2 copper layers, 100 x 85 mm, 70 parts, among them J1 USB_B_Mini, J10 Conn_01x10_Male, J11 Screw_Terminal_01x03, J12 Screw_Terminal_01x02, J2 Screw_Terminal_01x03, J3 Conn_01x04_Female, J4 57PC5FS, J5 Conn_01x02_Female, J6 Screw_Terminal_01x03, J7 Screw_Terminal_01x03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

Commit message: -
Parts:
- removed G***: LOGO, StudiokiController:Aisler_Logo
- removed the J8 at (184.6, 86.4)
- removed U5: MAX31865AAP+T, StudiokiController:SOP65P777X199-20N
Routing:
- net Net-(C16-Pad2): track 0.00 -> 7.19 mm

Commit message: -
Routing:
- net Net-(C16-Pad2): track 7.19 -> 0.00 mm
Changed lines of the file:
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@@
     (thickness 1.6)
     (drawings 20)
-    (tracks 451)
+    (tracks 449)
     (zones 0)
     (modules 67)
-    (nets 81)
+    (nets 80)
   )
   (page A4)
@@
   (net 78 "Net-(J11-Pad1)")
   (net 79 "Net-(J2-Pad1)")
-  (net 80 "Net-(C16-Pad2)")
   (net_class Default "This is the default net class."
     (clearance 0.15)
@@
     (add_net LED3)
     (add_net "Net-(C1-Pad1)")
-    (add_net "Net-(C16-Pad2)")
     (add_net "Net-(C3-Pad2)")
     (add_net "Net-(D2-Pad2)")
@@
     (add_net USB_TX)
   )
+  (module Connector_USB:USB_Micro-B_Molex-105017-0001 (layer F.Cu)
+    (at 209.575 129.675)
+    (descr http://www.molex.com/pdm_docs/sd/1050170001_sd.pdf)
+    (tags "Micro-USB SMD Typ-B")
+    (attr smd)
+    (fp_text reference J1 (at -5.064 2.8885) (layer F.SilkS)
+      (effects (font (size 1 1) (thickness 0.15)))
+    )
+    (fp_text value USB_B_Mini (at 0.3 4.3375) (layer F.Fab)
+      (effects (font (size 1 1) (thickness 0.15)))
+    )
+    (fp_line (start -1.1 -2.1225) (end -1.1 -1.9125) (layer F.Fab) (width 0.1))
+    (fp_line (start -1.5 -2.1225) (end -1.5 -1.9125) (layer F.Fab) (width 0.1))
+    (fp_line (start -1.5 -2.1225) (end -1.1 -2.1225) (layer F.Fab) (width 0.1))
+    (fp_line (start -1.1 -1.9125) (end -1.3 -1.7125) (layer F.Fab) (width 0.1))
+    (fp_line (start -1.3 -1.7125) (end -1.5 -1.9125) (layer F.Fab) (width 0.1))
+    (fp_line (start -1.7 -2.3125) (end -1.7 -1.8625) (layer F.SilkS) (width 0.12))
+    (fp_line (start -1.7 -2.3125) (end -1.25 -2.3125) (layer F.SilkS) (width 0.12))
+    (fp_line (start 3.9 -1.7625) (end 3.45 -1.7625) (layer F.SilkS) (width 0.12))
+    (fp_line (start 3.9 0.0875) (end 3.9 -1.7625) (layer F.SilkS) (width 0.12))
+    (fp_line (start -3.9 2.6375) (end -3.9 2.3875) (layer F.SilkS) (width 0.12))
+    (fp_line (start -3.75 3.3875) (end -3.75 -1.6125) (layer F.Fab) (width 0.1))
+    (fp_line (start -3.75 -1.6125) (end 3.75 -1.6125) (layer F.Fab) (width 0.1))
+    (fp_line (start -3.75 3.389204) (end 3.75 3.389204) (layer F.Fab) (width 0.1))
+    (fp_line (start -3 2.689204) (end 3 2.689204) (layer F.Fab) (width 0.1))
+    (fp_line (start 3.75 3.3875) (end 3.75 -1.6125) (layer F.Fab) (width 0.1))
+    (fp_line (start 3.9 2.6375) (end 3.9 2.3875) (layer F.SilkS) (width 0.12))
+    (fp_line (start -3.9 0.0875) (end -3.9 -1.7625) (layer F.SilkS) (width 0.12))
+    (fp_line (start -3.9 -1.7625) (end -3.45 -1.7625) (layer F.SilkS) (width 0.12))
+    (fp_line (start -4.4 3.64) (end -4.4 -2.46) (layer F.CrtYd) (width 0.05))
+    (fp_line (start -4.4 -2.46) (end 4.4 -2.46) (layer F.CrtYd) (width 0.05))
+    (fp_line (start 4.4 -2.46) (end 4.4 3.64) (layer F.CrtYd) (width 0.05))
+    (fp_line (start -4.4 3.64) (end 4.4 3.64) (layer F.CrtYd) (width 0.05))
+    (fp_text user %R (at 0 0.8875) (layer F.Fab)
+      (effects (font (size 1 1) (thickness 0.15)))
+    )
+    (fp_text user "PCB Edge" (at 0 2.6875) (layer Dwgs.User)
+      (effects (font (size 0.5 0.5) (thickness 0.08)))
+    )
+    (pad 6 smd rect (at -2.9 1.2375) (size 1.2 1.9) (layers F.Cu F.Mask)
+      (net 1 GND))
+    (pad 6 smd rect (at 2.9 1.2375) (size 1.2 1.9) (layers F.Cu F.Mask)
+      (net 1 GND))
+    (pad 6 thru_hole oval (at 3.5 1.2375) (size 1.2 1.9) (drill oval 0.6 1.3) (layers *.Cu *.Mask)
+      (net 1 GND))
+    (pad 6 thru_hole oval (at -3.5 1.2375 180) (size 1.2 1.9) (drill oval 0.6 1.3) (layers *.Cu *.Mask)
+      (net 1 GND))
+    (pad 6 smd rect (at -1 1.2375) (size 1.5 1.9) (layers F.Cu F.Paste F.Mask)
+      (net 1 GND))
+    (pad 6 thru_hole circle (at 2.5 -1.4625) (size 1.45 1.45) (drill 0.85) (layers *.Cu *.Mask)
+      (net 1 GND))
+    (pad 3 smd rect (at 0 -1.4625) (size 0.4 1.35) (layers F.Cu F.Paste F.Mask)
+      (net 23 "Net-(J1-Pad3)"))
+    (pad 4 smd rect (at 0.65 -1.4625) (size 0.4 1.35) (layers F.Cu F.Paste F.Mask)
+      (net 37 "Net-(J1-Pad4)"))
+    (pad 5 smd rect (at 1.3 -1.4625) (size 0.4 1.35) (layers F.Cu F.Paste F.Mask)
+      (net 1 GND))
+    (pad 1 smd rect (at -1.3 -1.4625) (size 0.4 1.35) (layers F.Cu F.Paste F.Mask)
+      (net 4 "Net-(C3-Pad2)"))
+    (pad 2 smd rect (at -0.65 -1.4625) (size 0.4 1.35) (layers F.Cu F.Paste F.Mask)
+      (net 22 "Net-(J1-Pad2)"))
+    (pad 6 thru_hole circle (at -2.5 -1.4625) (size 1.45 1.45) (drill 0.85) (layers *.Cu *.Mask)
+      (net 1 GND))
+    (pad 6 smd rect (at 1 1.2375) (size 1.5 1.9) (layers F.Cu F.Paste F.Mask)
+      (net 1 GND))
+    (model ${KISYS3DMOD}/Connector_USB.3dshapes/USB_Micro-B_Molex-105017-0001.wrl
+      (at (xyz 0 0 0))
+      (scale (xyz 1 1 1))
+      (rotate (xyz 0 0 0))
+    )
+  )
   (module RAC03-12SK:CONV_RAC03-12SK (layer F.Cu)
     (at 196.85 85.09)
@@
     )
   )
-  (module Connector_USB:USB_Micro-B_Molex-105017-0001 (layer F.Cu)
-    (at 209.575 129.675)
-    (descr http://www.molex.com/pdm_docs/sd/1050170001_sd.pdf)
-    (tags "Micro-USB SMD Typ-B")
-    (attr smd)
-    (fp_text reference J1 (at -5.064 2.8885) (layer F.SilkS)
-      (effects (font (size 1 1) (thickness 0.15)))
-    )
-    (fp_text value USB_B_Mini (at 0.3 4.3375) (layer F.Fab)
-      (effects (font (size 1 1) (thickness 0.15)))
-    )
-    (fp_line (start -1.1 -2.1225) (end -1.1 -1.9125) (layer F.Fab) (width 0.1))
-    (fp_line (start -1.5 -2.1225) (end -1.5 -1.9125) (layer F.Fab) (width 0.1))
-    (fp_line (start -1.5 -2.1225) (end -1.1 -2.1225) (layer F.Fab) (width 0.1))
-    (fp_line (start -1.1 -1.9125) (end -1.3 -1.7125) (layer F.Fab) (width 0.1))
-    (fp_line (start -1.3 -1.7125) (end -1.5 -1.9125) (layer F.Fab) (width 0.1))
-    (fp_line (start -1.7 -2.3125) (end -1.7 -1.8625) (layer F.SilkS) (width 0.12))
-    (fp_line (start -1.7 -2.3125) (end -1.25 -2.3125) (layer F.SilkS) (width 0.12))
-    (fp_line (start 3.9 -1.7625) (end 3.45 -1.7625) (layer F.SilkS) (width 0.12))
-    (fp_line (start 3.9 0.0875) (end 3.9 -1.7625) (layer F.SilkS) (width 0.12))
-    (fp_line (start -3.9 2.6375) (end -3.9 2.3875) (layer F.SilkS) (width 0.12))
-    (fp_line (start -3.75 3.3875) (end -3.75 -1.6125) (layer F.Fab) (width 0.1))
-    (fp_line (start -3.75 -1.6125) (end 3.75 -1.6125) (layer F.Fab) (width 0.1))
-    (fp_line (start -3.75 3.389204) (end 3.75 3.389204) (layer F.Fab) (width 0.1))
-    (fp_line (start -3 2.689204) (end 3 2.689204) (layer F.Fab) (width 0.1))
-    (fp_line (start 3.75 3.3875) (end 3.75 -1.6125) (layer F.Fab) (width 0.1))
-    (fp_line (start 3.9 2.6375) (end 3.9 2.3875) (layer F.SilkS) (width 0.12))
-    (fp_line (start -3.9 0.0875) (end -3.9 -1.7625) (layer F.SilkS) (width 0.12))
-    (fp_line (start -3.9 -1.7625) (end -3.45 -1.7625) (layer F.SilkS) (width 0.12))
-    (fp_line (start -4.4 3.64) (end -4.4 -2.46) (layer F.CrtYd) (width 0.05))
-    (fp_line (start -4.4 -2.46) (end 4.4 -2.46) (layer F.CrtYd) (width 0.05))
-    (fp_line (start 4.4 -2.46) (end 4.4 3.64) (layer F.CrtYd) (width 0.05))
-    (fp_line (start -4.4 3.64) (end 4.4 3.64) (layer F.CrtYd) (width 0.05))
-    (fp_text user %R (at 0 0.8875) (layer F.Fab)
-      (effects (font (size 1 1) (thickness 0.15)))
-    )
-    (fp_text user "PCB Edge" (at 0 2.6875) (layer Dwgs.User)
-      (effects (font (size 0.5 0.5) (thickness 0.08)))
-    )
-    (pad 6 smd rect (at -2.9 1.2375) (size 1.2 1.9) (layers F.Cu F.Mask)
-      (net 1 GND))
-    (pad 6 smd rect (at 2.9 1.2375) (size 1.2 1.9) (layers F.Cu F.Mask)
-      (net 1 GND))
-    (pad 6 thru_hole oval (at 3.5 1.2375) (size 1.2 1.9) (drill oval 0.6 1.3) (layers *.Cu *.Mask)
-      (net 1 GND))
-    (pad 6 thru_hole oval (at -3.5 1.2375 180) (size 1.2 1.9) (drill oval 0.6 1.3) (layers *.Cu *.Mask)
-      (net 1 GND))
-    (pad 6 smd rect (at -1 1.2375) (size 1.5 1.9) (layers F.Cu F.Paste F.Mask)
-      (net 1 GND))
-    (pad 6 thru_hole circle (at 2.5 -1.4625) (size 1.45 1.45) (drill 0.85) (layers *.Cu *.Mask)
-      (net 1 GND))
-    (pad 3 smd rect (at 0 -1.4625) (size 0.4 1.35) (layers F.Cu F.Paste F.Mask)
-      (net 23 "Net-(J1-Pad3)"))
-    (pad 4 smd rect (at 0.65 -1.4625) (size 0.4 1.35) (layers F.Cu F.Paste F.Mask)
-      (net 37 "Net-(J1-Pad4)"))
-    (pad 5 smd rect (at 1.3 -1.4625) (size 0.4 1.35) (layers F.Cu F.Paste F.Mask)
-      (net 1 GND))
-    (pad 1 smd rect (at -1.3 -1.4625) (size 0.4 1.35) (layers F.Cu F.Paste F.Mask)
-      (net 4 "Net-(C3-Pad2)"))
-    (pad 2 smd rect (at -0.65 -1.4625) (size 0.4 1.35) (layers F.Cu F.Paste F.Mask)
-      (net 22 "Net-(J1-Pad2)"))
-    (pad 6 thru_hole circle (at -2.5 -1.4625) (size 1.45 1.45) (drill 0.85) (layers *.Cu *.Mask)
-      (net 1 GND))
-    (pad 6 smd rect (at 1 1.2375) (size 1.5 1.9) (layers F.Cu F.Paste F.Mask)
-      (net 1 GND))
-    (model ${KISYS3DMOD}/Connector_USB.3dshapes/USB_Micro-B_Molex-105017-0001.wrl
-      (at (xyz 0 0 0))
-      (scale (xyz 1 1 1))
-      (rotate (xyz 0 0 0))
-    )
-  )
   (module Capacitor_SMD:C_0603_1608Metric (layer F.Cu)
     (at 240.225 122.025 90)
@@
   (segment (start 249.629999 63.039797) (end 248.551799 64.117997) (width 2) (layer F.Cu) (net 77))
   (segment (start 249.629999 53.34) (end 249.629999 63.039797) (width 2) (layer F.Cu) (net 77))
-  (segment (start 196.714 109.764) (end 197.1635 109.3145) (width 0.25) (layer F.Cu) (net 80))
-  (segment (start 190.162 109.764) (end 196.714 109.764) (width 0.25) (layer F.Cu) (net 80))
   (zone (net 1) (net_name GND) (layer F.Cu) (hatch edge 0.508)
     (connect_pads (clearance 0.508))

Commit message: -
Parts:
- removed J8: Conn_01x04_Female, Connector_PinSocket_2.54mm:PinSocket_1x04_P2.54mm_Vertical
- F1: footprint StudiokiController:Littelfuse65800001009 -> JanSquare:Littelfuse65800001009
- J4: footprint StudiokiController:57PC5FS -> JanSquare:57PC5FS
- PS1: footprint RAC03-12SK:CONV_RAC03-12SK -> JanSquare:CONV_RAC03-12SK
- moved F1 25.3 mm to (204.7, 60.5)
- moved RV1 7.34 mm to (192.8, 62.8), turned to 0 degrees
- moved J2 5.00 mm to (184.6, 53.3)
- moved PS1 4.84 mm to (192.4, 87.0)
Connections:
- net SPI_SS renamed CS_K1
- F1 pad 1: 230V-L -> 230V-N
- F1 pad 2: Net-(F1-Pad2) -> 230V-N
- J2 pad 2: Net-(F1-Pad2) -> 230V-L
- RV1 pad 1: 230V-N -> 230V-L
- RV1 pad 2: Net-(F1-Pad2) -> 230V-N
Routing:
- net Net-(F1-Pad2): track 24.6 -> 0.00 mm
- net 230V-L: track 8.20 -> 28.8 mm
- net 230V-N: track 23.2 -> 33.0 mm
- net +12V: track 100.5 -> 104.9 mm
