File: RaspiV2/raspiV2/raspiV2.kicad_pcb (KiCad board)
At the start: 2 copper layers, 80 x 80 mm, 1 part, among them J3 Raspberry_Pi_2_3

Commit message: kk
Parts:
- added D1: LED, LED_SMD:LED_0603_1608Metric, F.Cu at (161.6, 106.1)
- added D2: 1N4148W-TP, Diode_SMD:D_SOD-123, F.Cu at (162.4, 108.8)
- added D3: LED, LED_SMD:LED_0603_1608Metric, F.Cu at (175.6, 106.2)
- added D4: 1N4148W-TP, Diode_SMD:D_SOD-123, F.Cu at (176.4, 108.8)
- added H1: MountingHole, MountingHole:MountingHole_2.7mm_M2.5_ISO7380_Pad, F.Cu at (114.8, 64.3)
- added H2: MountingHole, MountingHole:MountingHole_2.7mm_M2.5_ISO7380_Pad, F.Cu at (186.1, 64.2)
- added H3: MountingHole, MountingHole:MountingHole_2.7mm_M2.5_ISO7380_Pad, F.Cu at (115.0, 136.1)
- added H4: MountingHole, MountingHole:MountingHole_2.7mm_M2.5_ISO7380_Pad, F.Cu at (185.8, 135.8)
- added J10: SPI, Connector_PinSocket_2.54mm:PinSocket_1x05_P2.54mm_Vertical, F.Cu at (141.0, 68.8)
- added J11: Screw_Terminal_01x02, TerminalBlock_Phoenix:TerminalBlock_Phoenix_PT-1,5-2-5.0-H_1x02_P5.00mm_Horizontal, F.Cu at (179.4, 135.2)
- added J4: SPI, Connector_PinSocket_2.54mm:PinSocket_1x05_P2.54mm_Vertical, F.Cu at (127.2, 68.8)
- added J5: 57PC5FS, JanSquare:57PC5FS, F.Cu at (170.2, 60.5)
- added J6: Screw_Terminal_01x02, TerminalBlock_Phoenix:TerminalBlock_Phoenix_PT-1,5-2-5.0-H_1x02_P5.00mm_Horizontal, F.Cu at (167.7, 68.2)
- added J7: Screw_Terminal_01x02, TerminalBlock_Phoenix:TerminalBlock_Phoenix_PT-1,5-2-5.0-H_1x02_P5.00mm_Horizontal, F.Cu at (165.2, 135.2)
- added J8: SPI, Connector_PinSocket_2.54mm:PinSocket_1x05_P2.54mm_Vertical, F.Cu at (131.8, 68.8)
- added J9: SPI, Connector_PinSocket_2.54mm:PinSocket_1x05_P2.54mm_Vertical, F.Cu at (136.4, 68.8)
- added Q1: PMV20XNE, Package_TO_SOT_SMD:SOT-23, F.Cu at (157.7, 107.2)
- added Q2: PMV20XNE, Package_TO_SOT_SMD:SOT-23, F.Cu at (171.3, 107.2)
- added R1: 10k, Resistor_SMD:R_0603_1608Metric, F.Cu at (154.7, 107.2)
- added R2: 10k, Resistor_SMD:R_0603_1608Metric, F.Cu at (168.3, 107.2)
- added RLA1: OJE-SH-112HM_000, JanSquare:OJE-SH-112HM_000, F.Cu at (158.9, 111.8)
- added RLA2: OJE-SH-112HM_000, JanSquare:OJE-SH-112HM_000, F.Cu at (173.2, 111.8)
- added U1: MAX31855KASA, Package_SO:SOIC-8_3.9x4.9mm_P1.27mm, F.Cu at (170.3, 81.5)
- added U2: ChinaLM2596, JanSquare:LM2596-Chinamodule, F.Cu at (141.9, 107.2)
Connections:
- J3 pad 13: Net-(J3-Pad13) -> RELAY1
- J3 pad 37: Net-(J3-Pad37) -> RELAY2

Commit message: update
Parts:
- removed the J10 at (141.0, 68.8)
- removed the J4 at (127.2, 68.8)
- removed the J9 at (136.4, 68.8)
- added J1: Door, TerminalBlock_Phoenix:TerminalBlock_Phoenix_PT-1,5-2-5.0-H_1x02_P5.00mm_Horizontal, F.Cu at (184.2, 100.2)
- added J2: Heater, TerminalBlock_Phoenix:TerminalBlock_Phoenix_PT-1,5-2-5.0-H_1x02_P5.00mm_Horizontal, F.Cu at (184.2, 88.2)
- added J5: PJ-002BH-SMT-TR, JanSquare:CUI_PJ-002BH-SMT-TR, F.Cu at (134.6, 128.2)
- added J6: Conn_01x06_Male, Connector_PinHeader_2.54mm:PinHeader_1x06_P2.54mm_Vertical, F.Cu at (133.4, 62.8)
- added J7: Conn_01x06_Male, Connector_PinHeader_2.54mm:PinHeader_1x06_P2.54mm_Vertical, F.Cu at (138.1, 62.8)
- J8: value SPI -> Conn_01x06_Male; footprint Connector_PinSocket_2.54mm:PinSocket_1x05_P2.54mm_Vertical -> Connector_PinHeader_2.54mm:PinHeader_1x06_P2.54mm_Vertical
- moved J8 12.5 mm to (142.8, 62.8)
- moved U1 7.38 mm to (139.6, 100.2)
- moved D3 0.50 mm to (176.1, 106.2)
- moved D4 0.50 mm to (176.9, 108.8)
- moved Q2 0.50 mm to (171.8, 107.2)
- moved R2 0.50 mm to (168.8, 107.2)
- renumbered J11 to J10, J6 to J11, J7 to J4, J5 to J9, U2 to U1, U1 to U2
Connections:
- net Net-(J1-Pad2) renamed DOOR
- net Net-(J2-Pad2) renamed HEATER
- J3 pad 15: Net-(J3-Pad15) -> CS1
- J3 pad 16: Net-(J3-Pad16) -> CS2
- J3 pad 19: Net-(J10-Pad4) -> Net-(J3-Pad19)
- J3 pad 21: Net-(J10-Pad3) -> Net-(J3-Pad21)
- J3 pad 22: Net-(J3-Pad22) -> CS3
- J3 pad 23: Net-(J10-Pad5) -> Net-(J3-Pad23)
- J3 pad 32: Net-(J3-Pad32) -> CS_81855
- J3 pad 35: Net-(J3-Pad35) -> SPI_MISO
- J3 pad 38: Net-(J3-Pad38) -> SPI_MOSI
- J3 pad 40: Net-(J3-Pad40) -> SPI_CLK
- J8 pad 1: +3V3 -> GND
- J8 pad 2: GND -> +3V3
- J8 pad 3: Net-(J10-Pad3) -> SPI_MISO
- J8 pad 4: Net-(J10-Pad4) -> SPI_MOSI
- J8 pad 5: Net-(J10-Pad5) -> SPI_CLK
- U2 pad 5: Net-(U1-Pad5) -> SPI_CLK
- U2 pad 6: Net-(U1-Pad6) -> CS_81855
- U2 pad 7: Net-(U1-Pad7) -> SPI_MISO
Routing:
- net SPI_MISO: track 0.00 -> 112.8 mm, vias 0 -> 2
- net SPI_CLK: track 0.00 -> 106.5 mm, vias 0 -> 2
- net CS_81855: track 0.00 -> 81.4 mm, vias 0 -> 2
- net +12V: track 0.00 -> 79.4 mm
- net RELAY2: track 0.00 -> 79.2 mm, vias 0 -> 2
- net SPI_MOSI: track 0.00 -> 75.7 mm, vias 0 -> 2
- net +3V3: track 0.00 -> 63.0 mm
- net RELAY1: track 0.00 -> 58.6 mm, vias 0 -> 2
- net CS3: track 0.00 -> 51.0 mm, vias 0 -> 1
- net CS2: track 0.00 -> 38.6 mm, vias 0 -> 1
- net CS1: track 0.00 -> 38.1 mm, vias 0 -> 1
- net Net-(J11-Pad1): track 0.00 -> 17.9 mm
- net Net-(J11-Pad2): track 0.00 -> 16.0 mm
- net +5V: track 0.00 -> 14.1 mm
- net Net-(J10-Pad2): track 0.00 -> 10.6 mm
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- added copper zone on B.Cu, net GND
- added copper zone on F.Cu, net GND

Commit message: update
Parts:
- added C1: C, Capacitor_SMD:C_0603_1608Metric, F.Cu at (166.5, 81.2)
- added J12: Conn_01x04_Female, Connector_PinSocket_2.54mm:PinSocket_1x04_P2.54mm_Vertical, F.Cu at (149.2, 67.7)
- added J13: Conn_01x04_Female, Connector_PinSocket_2.54mm:PinSocket_1x04_P2.54mm_Vertical, F.Cu at (153.8, 67.7)
- added J14: Conn_02x05_Odd_Even, Connector_IDC:IDC-Header_2x05_P2.54mm_Vertical, F.Cu at (161.8, 96.8)
- moved H2 1.28 mm to (185.0, 65.0)
- moved Q2 1.24 mm to (170.6, 107.1)
- moved RLA2 1.24 mm to (171.9, 111.7)
- moved J10 1.24 mm to (178.2, 135.2)
- moved D3 1.24 mm to (174.9, 106.1)
- moved D4 1.24 mm to (175.7, 108.8)
- moved R2 1.24 mm to (167.6, 107.2)
- moved U1 1.15 mm to (139.7, 101.4)
- moved H4 1.10 mm to (185.0, 135.0)
- moved H3 1.04 mm to (115.0, 135.0)
- moved H1 0.68 mm to (115.0, 65.0)
Connections:
- J1 pad 1: Net-(J1-Pad1) -> GND
- J1 pad 2: Net-(J1-Pad2) -> DOOR
- J2 pad 1: Net-(J2-Pad1) -> GND
- J2 pad 2: Net-(J2-Pad2) -> HEATER
- J3 pad 19: Net-(J3-Pad19) -> SPI_MOSI
- J3 pad 21: Net-(J3-Pad21) -> SPI_MISO
- J3 pad 23: Net-(J3-Pad23) -> SPI_CLK
- J3 pad 24: Net-(J3-Pad24) -> GPIO_8
- J3 pad 26: Net-(J3-Pad26) -> GPIO_7
- J3 pad 27: Net-(J3-Pad27) -> GPIO_0
- J3 pad 28: Net-(J3-Pad28) -> GPIO_1
- J3 pad 29: Net-(J3-Pad29) -> GPIO_5
- J3 pad 3: Net-(J3-Pad3) -> SDA
- J3 pad 31: Net-(J3-Pad31) -> GPIO_6
- J3 pad 35: SPI_MISO -> Net-(J3-Pad35)
- J3 pad 38: SPI_MOSI -> Net-(J3-Pad38)
- J3 pad 40: SPI_CLK -> Net-(J3-Pad40)
- J3 pad 5: Net-(J3-Pad5) -> SCL
- J3 pad 7: Net-(J3-Pad7) -> GPIO_4
Routing:
- net GPIO_8: track 0.00 -> 71.2 mm, vias 0 -> 3
- net HEATER: track 0.00 -> 70.3 mm
- net GPIO_6: track 0.00 -> 69.8 mm, vias 0 -> 3
- net GPIO_7: track 0.00 -> 68.7 mm, vias 0 -> 3
- net DOOR: track 0.00 -> 66.9 mm
- net GPIO_5: track 0.00 -> 66.1 mm, vias 0 -> 3
- net GPIO_4: track 0.00 -> 63.3 mm, vias 0 -> 1
- net GPIO_1: track 0.00 -> 61.2 mm, vias 0 -> 3
- net GPIO_0: track 0.00 -> 61.0 mm, vias 0 -> 3
- net SCL: track 0.00 -> 48.5 mm, vias 0 -> 1
- net +3V3: track 63.0 -> 110.7 mm, vias 0 -> 1
- net SDA: track 0.00 -> 42.1 mm
- net SPI_MOSI: track 75.7 -> 55.0 mm
- net SPI_MISO: track 112.8 -> 102.4 mm, vias 2 -> 4
- net SPI_CLK: track 106.5 -> 96.4 mm, vias 2 -> 4
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Other:
- board text added: "0"
- board text added: "1"
- board text added: "3V3"
- board text added: "4"
- board text added: "5"
- board text added: "6"
- board text added: "7"
- board text added: "8"
- board text added: "CLK"
- board text added: "CS1"
- board text added: "CS2"
- board text added: "CS3"
- board text added: "GND"
- board text added: "MISO"
- board text added: "MOSI"
- board text added: "SCL"
- board text added: "SDA"

Commit message: minor changes
Parts:
- J3: value Raspberry_Pi_2_3 -> PPTC202LFBN-RC
Changed lines of the file:
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@@
   )
   (setup
-    (last_trace_width 0.8)
+    (last_trace_width 0.25)
     (user_trace_width 0.8)
     (user_trace_width 1.2)
@@
       (effects (font (size 1 1) (thickness 0.15)))
     )
-    (fp_text value Raspberry_Pi_2_3 (at 1.27 50.59) (layer F.Fab)
-      (effects (font (size 1 1) (thickness 0.15)))
-    )
+    (fp_text value PPTC202LFBN-RC (at 1.27 50.59) (layer F.Fab)
+      (effects (font (size 1 1) (thickness 0.15)))
+    )
