File: RaspiV2/raspiV2/raspiV2.sch (KiCad schematic (older format))
At the start: 4 parts, among them J1 Door, J2 Heater, J3 Raspberry_Pi_2_3, J4 SPI

Commit message: kk
Parts:
- added D1, D3: LED, LED_SMD:LED_0603_1608Metric, symbol Device:LED
- added D2, D4: 1N4148W-TP, Diode_SMD:D_SOD-123, symbol Device:D
- added H1, H2, H3, H4: MountingHole, MountingHole:MountingHole_2.7mm_M2.5_ISO7380_Pad, symbol Mechanical:MountingHole
- added J10, J8, J9: SPI, Connector_PinSocket_2.54mm:PinSocket_1x05_P2.54mm_Vertical, symbol Connector:Conn_01x05_Male
- added J11, J6, J7: Screw_Terminal_01x02, TerminalBlock_Phoenix:TerminalBlock_Phoenix_PT-1,5-2-5.0-H_1x02_P5.00mm_Horizontal, symbol Connector:Screw_Terminal_01x02
- added J5: 57PC5FS, 57PC5FS, symbol JanSquareLib:57PC5FS
- added Q1, Q2: PMV20XNE, Package_TO_SOT_SMD:SOT-23, symbol Device:Q_NMOS_GSD
- added R1, R2: 10k, Resistor_SMD:R_0603_1608Metric, symbol Device:R
- added RLA1, RLA2: OJE-SH-112HM_000, JanSquare:OJE-SH-112HM_000, symbol JanSquareLib:OJE-SH-112HM_000
- added U1: MAX31855KASA, Package_SO:SOIC-8_3.9x4.9mm_P1.27mm, symbol Sensor_Temperature:MAX31855KASA
- added U2: ChinaLM2596, JanSquare:LM2596-Chinamodule, symbol JanSquareLib:ChinaLM2596
- J4: footprint (none) -> Connector_PinSocket_2.54mm:PinSocket_1x05_P2.54mm_Vertical
Connections:
- net +3V3: now also J10.1 (Pin_1), J8.1 (Pin_1), J9.1 (Pin_1), U1.4 (VCC)
- net +5V: now also U2.3 (+OUT)
- net GND: now also D1.1 (K), D3.1 (K), J10.2 (Pin_2), J5.6 (GROUND_1), J5.7 (GROUND_2), J8.2 (Pin_2), J9.2 (Pin_2), Q1.2 (S), Q2.2 (S), R1.2, R2.2, U1.1 (GND), U2.2 (-IN), U2.4 (-OUT)
- net RELAY1: now reaches J3.13 (GPIO27)
- net RELAY1: now also D1.2 (A), Q1.1 (G), R1.1
- net at J3.19 (MOSI0/GPIO10), J4.4 (Pin_4): now also J10.4 (Pin_4), J8.4 (Pin_4), J9.4 (Pin_4)
- net at J3.21 (MISO0/GPIO9), J4.3 (Pin_3): now also J10.3 (Pin_3), J8.3 (Pin_3), J9.3 (Pin_3)
- net at J3.23 (SCLK0/GPIO11), J4.5 (Pin_5): now also J10.5 (Pin_5), J8.5 (Pin_5), J9.5 (Pin_5)
- net RELAY2: now reaches J3.37 (GPIO26)
- net RELAY2: now also D3.2 (A), Q2.1 (G), R2.1
- new net: J7.1 (Pin_1), RLA1.1
- new net: D2.2 (A), Q1.3 (D), RLA1.3
- new net: J7.2 (Pin_2), RLA1.4
- new net: J11.1 (Pin_1), RLA2.1
- new net: J11.2 (Pin_2), RLA2.4
- new net: D4.2 (A), Q2.3 (D), RLA2.3
- new net: J5.3, J6.2 (Pin_2), U1.2 (T-)
- new net: J5.1, J6.1 (Pin_1), U1.3 (T+)
- new net +12V: D2.1 (K), D4.1 (K), RLA1.2, RLA2.2, U2.1 (+IN)
- no-connect marks 0 -> 3
Other:
- moved on the sheet: J1, J2, J3, J4

Commit message: update
Parts:
- removed J10, J4, J8, J9: SPI, Connector_PinSocket_2.54mm:PinSocket_1x05_P2.54mm_Vertical, symbol Connector:Conn_01x05_Male
- added J5: PJ-002BH-SMT-TR, CUI_PJ-002BH-SMT-TR, symbol JanSquareLib:PJ-002BH-SMT-TR
- added J6, J7, J8: Conn_01x06_Male, Connector_PinHeader_2.54mm:PinHeader_1x06_P2.54mm_Vertical, symbol Connector:Conn_01x06_Male
- J1, J2: footprint (none) -> TerminalBlock_Phoenix:TerminalBlock_Phoenix_PT-1,5-2-5.0-H_1x02_P5.00mm_Horizontal
- renumbered J11 to J10, J6 to J11, J7 to J4, J5 to J9, U2 to U1, U1 to U2
Connections:
- net +12V: now also J5.1A (1), J5.1B (1)
- net +3V3: now also J6.2 (Pin_2), J7.2 (Pin_2), J8.2 (Pin_2)
- net GND: now also J5.2, J6.1 (Pin_1), J7.1 (Pin_1), J8.1 (Pin_1)
- net at J2.2 (Pin_2): no longer J3.11 (GPIO17)
- net CS1: now reaches J3.15 (GPIO22)
- net CS1: now also J6.6 (Pin_6)
- net CS2: now reaches J3.16 (GPIO23)
- net CS2: now also J7.6 (Pin_6)
- net at J1.2 (Pin_2): no longer J3.18 (GPIO24)
- net CS3: now reaches J3.22 (GPIO25)
- net CS3: now also J8.6 (Pin_6)
- net CS_81855: now reaches J3.32 (PWM0/GPIO12)
- net CS_81855: now also U2.6 (~CS~)
- net SPI_MISO: now reaches J3.35 (GPIO19/MISO1)
- net SPI_MISO: now also U2.7 (SO), J6.3 (Pin_3), J7.3 (Pin_3), J8.3 (Pin_3)
- net SPI_MOSI: now reaches J3.38 (GPIO20/MOSI1)
- net SPI_MOSI: now also J6.4 (Pin_4), J7.4 (Pin_4), J8.4 (Pin_4)
- net SPI_CLK: now reaches J3.40 (GPIO21/SCLK1)
- net SPI_CLK: now also U2.5 (SCK), J6.5 (Pin_5), J7.5 (Pin_5), J8.5 (Pin_5)
- new net DOOR: J3.18 (GPIO24)
- new net HEATER: J3.11 (GPIO17)
Other:
- note added: "12V IN --> 5V"
- moved on the sheet: H1, H2, H3, H4, J1, J2, U1

Commit message: update
Parts:
- added C1: C, Capacitor_SMD:C_0603_1608Metric, symbol Device:C
- added J12, J13: Conn_01x04_Female, Connector_PinSocket_2.54mm:PinSocket_1x04_P2.54mm_Vertical, symbol Connector:Conn_01x04_Female
- added J14: Conn_02x05_Odd_Even, Connector_IDC:IDC-Header_2x05_P2.54mm_Vertical, symbol Connector_Generic:Conn_02x05_Odd_Even
Connections:
- net +3V3: now also C1.1, J12.2 (Pin_2), J13.2 (Pin_2), J14.1 (Pin_1)
- net DOOR: now also J1.2 (Pin_2)
- net GND: now also J1.1 (Pin_1), J2.1 (Pin_1), C1.2, J12.1 (Pin_1), J13.1 (Pin_1), J14.2 (Pin_2), J14.7 (Pin_7)
- net HEATER: now also J2.2 (Pin_2)
- net SPI_CLK: now also J3.23 (SCLK0/GPIO11); no longer J3.40 (GPIO21/SCLK1)
- net SPI_MISO: now also J3.21 (MISO0/GPIO9); no longer J3.35 (GPIO19/MISO1)
- net SPI_MOSI: now also J3.19 (MOSI0/GPIO10); no longer J3.38 (GPIO20/MOSI1)
- net GPIO_8: now reaches J3.24 (~CE0~/GPIO8)
- net GPIO_8: now also J14.10 (Pin_10)
- net GPIO_7: now reaches J3.26 (~CE1~/GPIO7)
- net GPIO_7: now also J14.8 (Pin_8)
- net GPIO_0: now reaches J3.27 (ID_SD/GPIO0)
- net GPIO_0: now also J14.3 (Pin_3)
- net GPIO_1: now reaches J3.28 (ID_SC/GPIO1)
- net GPIO_1: now also J14.5 (Pin_5)
- net GPIO_5: now reaches J3.29 (GCLK1/GPIO5)
- net GPIO_5: now also J14.4 (Pin_4)
- net SDA: now reaches J3.3 (SDA/GPIO2)
- net SDA: now also J12.4 (Pin_4), J13.4 (Pin_4)
- net GPIO_6: now reaches J3.31 (GCLK2/GPIO6)
- net GPIO_6: now also J14.6 (Pin_6)
- net SCL: now reaches J3.5 (SCL/GPIO3)
- net SCL: now also J12.3 (Pin_3), J13.3 (Pin_3)
- net GPIO_4: now reaches J3.7 (GCLK0/GPIO4)
- net GPIO_4: now also J14.9 (Pin_9)
Other:
- moved on the sheet: J1, J2
Changed lines of the file:
@@
 L Connector:Conn_01x02_Male J2
 U 1 1 5E4FABA1
-P 4350 2500
-F 0 "J2" H 4458 2681 50  0000 C CNN
-F 1 "Heater" H 4458 2590 50  0000 C CNN
-F 2 "TerminalBlock_Phoenix:TerminalBlock_Phoenix_PT-1,5-2-5.0-H_1x02_P5.00mm_Horizontal" H 4350 2500 50  0001 C CNN
-F 3 "~" H 4350 2500 50  0001 C CNN
-	1    4350 2500
+P 4150 1750
+F 0 "J2" H 4258 1931 50  0000 C CNN
+F 1 "Heater" H 4258 1840 50  0000 C CNN
+F 2 "TerminalBlock_Phoenix:TerminalBlock_Phoenix_PT-1,5-2-5.0-H_1x02_P5.00mm_Horizontal" H 4150 1750 50  0001 C CNN
+F 3 "~" H 4150 1750 50  0001 C CNN
+	1    4150 1750
 	1    0    0    -1
 $EndComp
@@
 L Connector:Conn_01x02_Male J1
 U 1 1 5E4FB99A
-P 4350 2900
-F 0 "J1" H 4458 3081 50  0000 C CNN
-F 1 "Door" H 4458 2990 50  0000 C CNN
-F 2 "TerminalBlock_Phoenix:TerminalBlock_Phoenix_PT-1,5-2-5.0-H_1x02_P5.00mm_Horizontal" H 4350 2900 50  0001 C CNN
-F 3 "~" H 4350 2900 50  0001 C CNN
-	1    4350 2900
+P 4150 2150
+F 0 "J1" H 4258 2331 50  0000 C CNN
+F 1 "Door" H 4258 2240 50  0000 C CNN
+F 2 "TerminalBlock_Phoenix:TerminalBlock_Phoenix_PT-1,5-2-5.0-H_1x02_P5.00mm_Horizontal" H 4150 2150 50  0001 C CNN
+F 3 "~" H 4150 2150 50  0001 C CNN
+	1    4150 2150
 	1    0    0    -1
 $EndComp
@@
 	8900 3200 9150 3200
 Connection ~ 9150 3200
-Text GLabel 1600 2400 0    50   Input ~ 0
+Text GLabel 3200 2900 2    50   Input ~ 0
 SPI_MISO
-Text GLabel 1600 2500 0    50   Input ~ 0
+Text GLabel 3200 3000 2    50   Input ~ 0
 SPI_MOSI
-Text GLabel 1600 2600 0    50   Input ~ 0
+Text GLabel 3200 3100 2    50   Input ~ 0
 SPI_CLK
 Text Notes 10050 900  2    50   ~ 0
 12V IN --> 5V
 $Comp
-L power:GND #PWR?
+L power:GND #PWR0101
 U 1 1 5E596F13
 P 10350 6150
-F 0 "#PWR?" H 10350 5900 50  0001 C CNN
+F 0 "#PWR0101" H 10350 5900 50  0001 C CNN
 F 1 "GND" H 10355 5977 50  0000 C CNN
 F 2 "" H 10350 6150 50  0001 C CNN
@@
 Text GLabel 3200 3300 2    50   Input ~ 0
 CS_81855
+Text GLabel 3200 2000 2    50   Input ~ 0
+SDA
+Text GLabel 3200 2100 2    50   Input ~ 0
+SCL
+$Comp
+L Connector:Conn_01x04_Female J12
+U 1 1 5E5CC3B8
+P 3800 950
+F 0 "J12" H 3828 926 50  0000 L CNN
+F 1 "Conn_01x04_Female" H 3828 835 50  0000 L CNN
+F 2 "Connector_PinSocket_2.54mm:PinSocket_1x04_P2.54mm_Vertical" H 3800 950 50  0001 C CNN
+F 3 "~" H 3800 950 50  0001 C CNN
+	1    3800 950
+	1    0    0    -1
+$EndComp
+Text GLabel 3600 1150 0    50   Input ~ 0
+SDA
+Text GLabel 3600 1050 0    50   Input ~ 0
+SCL
+$Comp
+L power:GND #PWR0103
+U 1 1 5E5D113A
+P 3600 850
+F 0 "#PWR0103" H 3600 600 50  0001 C CNN
+F 1 "GND" H 3605 677 50  0000 C CNN
+F 2 "" H 3600 850 50  0001 C CNN
+F 3 "" H 3600 850 50  0001 C CNN
+	1    3600 850
+	0    1    1    0
+$EndComp
+$Comp
+L Connector:Conn_01x04_Female J13
+U 1 1 5E5D4F02
+P 4150 950
+F 0 "J13" H 4178 926 50  0000 L CNN
+F 1 "Conn_01x04_Female" H 4178 835 50  0000 L CNN
+F 2 "Connector_PinSocket_2.54mm:PinSocket_1x04_P2.54mm_Vertical" H 4150 950 50  0001 C CNN
+F 3 "~" H 4150 950 50  0001 C CNN
+	1    4150 950
+	1    0    0    -1
+$EndComp
+Wire Wire Line
+	3600 850  3950 850
+Connection ~ 3600 850
+Wire Wire Line
+	3600 950  3950 950
+Wire Wire Line
+	3600 1050 3950 1050
+Wire Wire Line
+	3600 1150 3950 1150
+Text GLabel 3200 1700 2    50   Input ~ 0
+GPIO_0
+Text GLabel 3200 1800 2    50   Input ~ 0
+GPIO_1
+Text GLabel 3200 2300 2    50   Input ~ 0
+GPIO_4
+Text GLabel 3200 2400 2    50   Input ~ 0
+GPIO_5
+Text GLabel 3200 2500 2    50   Input ~ 0
+GPIO_6
+Text GLabel 3200 2700 2    50   Input ~ 0
+GPIO_7
+Text GLabel 3200 2800 2    50   Input ~ 0
+GPIO_8
+$Comp
+L power:GND #PWR0104
+U 1 1 5E5ED1A4
+P 4350 1750
+F 0 "#PWR0104" H 4350 1500 50  0001 C CNN
+F 1 "GND" H 4355 1577 50  0000 C CNN
+F 2 "" H 4350 1750 50  0001 C CNN
+F 3 "" H 4350 1750 50  0001 C CNN
+	1    4350 1750
+	0    -1   -1   0
+$EndComp
+$Comp
+L power:GND #PWR0105
+U 1 1 5E5EDB39
+P 4350 2150
+F 0 "#PWR0105" H 4350 1900 50  0001 C CNN
+F 1 "GND" H 4355 1977 50  0000 C CNN
+F 2 "" H 4350 2150 50  0001 C CNN
+F 3 "" H 4350 2150 50  0001 C CNN
+	1    4350 2150
+	0    -1   -1   0
+$EndComp
+Text GLabel 4350 2250 2    50   Input ~ 0
+DOOR
+Text GLabel 4350 1850 2    50   Input ~ 0
+HEATER
+$Comp
+L Connector_Generic:Conn_02x05_Odd_Even J14
+U 1 1 5E5F8338
+P 5300 3050
+F 0 "J14" H 5350 3467 50  0000 C CNN
+F 1 "Conn_02x05_Odd_Even" H 5350 3376 50  0000 C CNN
+F 2 "Connector_IDC:IDC-Header_2x05_P2.54mm_Vertical" H 5300 3050 50  0001 C CNN
+F 3 "~" H 5300 3050 50  0001 C CNN
+	1    5300 3050
+	1    0    0    -1
+$EndComp
+Text GLabel 5600 3250 2    50   Input ~ 0
+GPIO_8
+Text GLabel 5600 3150 2    50   Input ~ 0
+GPIO_7
+Text GLabel 5600 3050 2    50   Input ~ 0
+GPIO_6
+Text GLabel 5600 2950 2    50   Input ~ 0
+GPIO_5
+Text GLabel 5100 3250 0    50   Input ~ 0
+GPIO_4
+Text GLabel 5100 2950 0    50   Input ~ 0
+GPIO_0
+Text GLabel 5100 3050 0    50   Input ~ 0
+GPIO_1
+$Comp
+L power:GND #PWR0106
+U 1 1 5E5FEAB8
+P 5600 2850
+F 0 "#PWR0106" H 5600 2600 50  0001 C CNN
+F 1 "GND" H 5605 2677 50  0000 C CNN
+F 2 "" H 5600 2850 50  0001 C CNN
+F 3 "" H 5600 2850 50  0001 C CNN
+	1    5600 2850
+	0    -1   -1   0
+$EndComp
+$Comp
+L power:GND #PWR0107
+U 1 1 5E5FF166
+P 5100 3150
+F 0 "#PWR0107" H 5100 2900 50  0001 C CNN
+F 1 "GND" H 5105 2977 50  0000 C CNN
+F 2 "" H 5100 3150 50  0001 C CNN
+F 3 "" H 5100 3150 50  0001 C CNN
+	1    5100 3150
+	0    1    1    0
+$EndComp
+$Comp
+L power:+3.3V #PWR0108
+U 1 1 5E600374
+P 5100 2850
+F 0 "#PWR0108" H 5100 2700 50  0001 C CNN
+F 1 "+3.3V" H 5115 3023 50  0000 C CNN
+F 2 "" H 5100 2850 50  0001 C CNN
+F 3 "" H 5100 2850 50  0001 C CNN
+	1    5100 2850
+	0    -1   -1   0
+$EndComp
+$Comp
+L power:+3.3V #PWR0102
+U 1 1 5E609A94
+P 3600 950
+F 0 "#PWR0102" H 3600 800 50  0001 C CNN
+F 1 "+3.3V" H 3615 1123 50  0000 C CNN
+F 2 "" H 3600 950 50  0001 C CNN
+F 3 "" H 3600 950 50  0001 C CNN
+	1    3600 950
+	0    -1   -1   0
+$EndComp
+Connection ~ 3600 950
+$Comp
+L Device:C C1
+U 1 1 5E61C5A6
+P 8750 1500
+F 0 "C1" H 8865 1546 50  0000 L CNN
+F 1 "C" H 8865 1455 50  0000 L CNN
+F 2 "Capacitor_SMD:C_0603_1608Metric" H 8788 1350 50  0001 C CNN
+F 3 "~" H 8750 1500 50  0001 C CNN
+	1    8750 1500
+	1    0    0    -1
+$EndComp
+Wire Wire Line
+	7800 1100 8750 1100
+Wire Wire Line
+	8750 1100 8750 1350
+Connection ~ 7800 1100
+Wire Wire Line
+	7800 1900 8750 1900
+Wire Wire Line
+	8750 1650 8750 1900
+Connection ~ 7800 1900
 $EndSCHEMATC
